Commit message: Forward kinematics finished

File: rrm_cv3_trebula/urdf/arm.urdf (robot description, URDF)
Before this commit: robot arm, 11 links, 10 joints
Joints:
- removed joint joint_3b
- removed joint link3_to_joint_3b
- added joint joint_3: type prismatic, parent joint_3a, child joint_3b, origin xyz=0 0 0 rpy=0 0 0, axis 0 0 1, limit lower=0.0 upper=0.10 effort=1000.0 velocity=0.5
- added joint joint_3b_to_link3: type fixed, parent joint_3b, child link3, origin xyz=0 0 0.081 rpy=0 0 0
- joint joint_4_to_tool0: origin xyz=0 0 0.11 rpy=0 0 0 -> xyz=0 0 0.08 rpy=0 0 0
- joint link2_to_joint_3a: origin xyz=0 0 0.09 rpy=0 0 0 -> xyz=0 0 0.081 rpy=0 0 0
- joint link4_to_joint_4: origin xyz=0 0 0.069 rpy=0 0 0 -> xyz=0 0 0.04 rpy=0 0 0

Commit message: forward kinematics updated

File: rrm_cv3_trebula/urdf/arm.urdf (robot description, URDF)
Before this commit: robot arm, 11 links, 10 joints
Joints:
- removed joint joint_3
- added joint joint_3b: type prismatic, parent joint_3a, child joint_3b, origin xyz=0 0 0 rpy=0 0 0, axis 0 0 1, limit lower=0.0 upper=0.10 effort=1000.0 velocity=0.5
