Commit message: Sensor added

File: abb_camera_simulation/urdf/abb_irb4600_60_205_macro.xacro (robot description, xacro)
@@ -263,5 +263,5 @@
             <parent link="${prefix}link_6"/>
             <child link="${prefix}tool0"/>
-            <origin xyz="0.135 0 0" rpy="0 1.570796 0"/>
+            <origin xyz="0.15 0 0" rpy="0 0 0"/>
         </joint>
         <joint name="to_kinect" type="fixed">
@@ -287,5 +287,5 @@
             <child link="kinect_mesh"/>
             <limit lower="0" upper="0" effort="0" velocity="0"/>
-            <origin xyz="0 0 0.015" rpy="0 0 1.57"/>
+            <origin xyz="0 0 0" rpy="0 0 1.57"/>
         </joint>
         <link name ="kinect_frame"/>
